Commit message: Added test manipulator code

File: urdf/Test_urdf/manipulator.urdf (robot description, URDF)
Before this commit: robot manipulator, 4 links, 3 joints
Joints:
- joint Revolute 3: limit (none) -> lower=-3.141592653589793 upper=3.141592653589793 effort=3.1 velocity=8; type continuous -> revolute
- joint Revolute 4: limit (none) -> lower=-3.141592653589793 upper=3.141592653589793 effort=3.1 velocity=8; type continuous -> revolute
- joint Revolute 5: limit (none) -> lower=-3.141592653589793 upper=3.141592653589793 effort=3.1 velocity=8; type continuous -> revolute

Commit message: Fixed Test_urdf

File: urdf/Test_urdf/manipulator.urdf (robot description, URDF)
Before this commit: robot manipulator, 4 links, 3 joints
Joints:
- joint Revolute 4: axis -0.986777 -0.162084 -0.0 -> -0.999997 0.002434 0.0; origin xyz=-0.025737 -0.00372 0.0563 rpy=0 0 0 -> xyz=-0.025999 0.000564 0.0563 rpy=0 0 0
- joint Revolute 5: axis 0.986777 0.162084 0.0 -> 0.999997 -0.002434 0.0; origin xyz=0.029825 0.136161 0.09444 rpy=0 0 0 -> xyz=0.051496 -0.00191 0.160291 rpy=0 0 0

Commit message: Added real time control

File: urdf/Test_urdf/manipulator.urdf (robot description, URDF)
Before this commit: robot manipulator, 4 links, 3 joints
Links:
- added link end_eff
Joints:
- added joint joint_ee: type fixed, parent link_3_v4_1, child end_eff, origin xyz=-0.0255 0.00 0.09 rpy=0 0 0
- joint Revolute 3: axis -0.0 -0.0 1.0 -> -0.0 -0.0 -1.0
- joint Revolute 4: axis -0.999997 0.002434 0.0 -> 0.999997 -0.002434 0.0
